File: pcb/Clankerplant/Clankerplant.kicad_sch (KiCad schematic)
At the start: 0 parts

Commit message: backup incase deleitng stuff goes wrong
Parts:
- added C1, C5: 1uF, symbol Device:C
- added C10, C11: TBD, symbol Device:C
- added C2, C6, C9: 10uF, symbol Device:C
- added C3, C4, C7, C8: 0.1uF, symbol Device:C
- added D1: ESD, symbol Device:D_TVS
- added J1: flash, symbol Connector:Conn_01x06_Socket
- added J3: LCD screen, Connector_PinHeader_2.54mm:PinHeader_1x07_P2.54mm_Vertical, symbol Connector_Generic:Conn_01x07
- added J4: water pump, Connector_PinHeader_2.54mm:PinHeader_1x02_P2.54mm_Vertical, symbol Connector_Generic:Conn_01x02
- added L1: 2.0nH, symbol Device:L
- added L2: 24 nH, symbol Device:L
- added Q2: AO3400A (mosfet), Package_TO_SOT_SMD:SOT-23, symbol Transistor_FET:AO3400A
- added R2: 499, symbol Device:R_US
- added U2: ESP32-S3, Package_DFN_QFN:QFN-56-1EP_7x7mm_P0.4mm_EP4x4mm, symbol MCU_Espressif:ESP32-S3
- added Y1: 40MHz, symbol Device:Crystal_GND24
Connections:
- new net: C11.2, U2.53 (XTAL_N), Y1.3
- new net: C3.1, L1.1, U2.2 (VDD3P3), U2.3 (VDD3P3)
- new net: C10.2, L2.1, Y1.1
- new net: L2.2, U2.54 (XTAL_P)
- new net: R2.2, U2.50 (U0RXD)
- new net +3.3V: C1.1, C2.1, C4.1, C5.1, C6.1, L1.2, U2.55 (VDDA), U2.56 (VDDA)
- new net +3V3: C7.1, C8.1, C9.1, D1.2 (A2), J1.1 (Pin_1), U2.20 (VDD3P3_RTC), U2.46 (VDD3P3_CPU)
- new net CHIP_EN: J1.5 (Pin_5), U2.4 (CHIP_PU)
- new net CS: J3.CS
- new net DC: J3.DC
- new net GND: C1.2, C10.1, C11.1, C2.2, C3.2, C4.2, C5.2, C6.2, C7.2, C8.2, C9.2, D1.1 (A1), J1.2 (Pin_2), J3.GND, J4.GND, U2.57 (GND), Y1.2 (G), Y1.4 (G)
- new net GPIO1: U2.6 (GPIO1)
- new net GPIO10: U2.15 (GPIO10)
- new net GPIO11: U2.16 (GPIO11)
- new net GPIO12: U2.17 (GPIO12)
- new net GPIO13: U2.18 (GPIO13)
- new net GPIO14: U2.19 (GPIO14)
- new net GPIO17: U2.23 (GPIO17)
- new net GPIO18: U2.24 (GPIO18)
- new net GPIO2: U2.7 (GPIO2)
- new net GPIO3: U2.8 (GPIO3)
- new net GPIO4: U2.9 (GPIO4)
- new net GPIO5: U2.10 (GPIO5)
- new net GPIO6: U2.11 (GPIO6)
- new net GPIO7: U2.12 (GPIO7)
- new net GPIO8: U2.13 (GPIO8)
- new net GPIO9: J1.6 (Pin_6), U2.14 (GPIO9)
- new net LCD_VCC: J3.VCC
- new net PUMP_PWR: J4.PWR
- new net RST: J3.RST
- new net SCL: J3.SCL
- new net SDA: J3.SDA
- new net U0RXD: J1.3 (Pin_3), U2.49 (U0TXD)
- new net U0TXD: J1.4 (Pin_4), R2.1
- no-connect marks 0 -> 29
Other:
- note added: "batt"
- note added: "mcu"
- note added: "sensors"
- title: (none) -> clankerplant
