File: pcb/penguinplant/penguinplant.kicad_pcb (KiCad board)
At the start: 2 copper layers, 41.7 x 34.6 mm, 8 parts, among them J1 Soil Sensor, J2 pump, J3 LCD, Q1 AO3400, U2 XIAO-nRF52840-SMD

Commit message: silkscreen
Parts:
- added G***: LOGO, LOGO, B.Cu at (140.2, 104.8)
- added G***: LOGO, LOGO, B.Cu at (152.2, 109.2)
- added G***: LOGO, LOGO, B.Cu at (141.0, 112.4)
Other:
- board text added: "penguinplant"
